File: UccMicroDuino/UccMicroDuino.kicad_sch (KiCad schematic)
At the start: 14 parts, among them J2 PCB USB Type A, J2 header, U2 ATtiny85-20S

Commit message: Add files via upload
Parts:
- D4: footprint (none) -> ledSmd:ledSMD
- R2, R3: footprint (none) -> Resistor_SMD:R_0805_2012Metric_Pad1.20x1.40mm_HandSolder
Changed lines of the file:
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@@
 			)
 		)
-		(property "Footprint" ""
+		(property "Footprint" "Resistor_SMD:R_0805_2012Metric_Pad1.20x1.40mm_HandSolder"
 			(at 256.032 87.63 90)
 			(effects
@@
 			)
 		)
-		(property "Footprint" ""
+		(property "Footprint" "ledSmd:ledSMD"
 			(at 179.07 77.47 0)
 			(effects
@@
 			)
 		)
-		(property "Footprint" ""
+		(property "Footprint" "Resistor_SMD:R_0805_2012Metric_Pad1.20x1.40mm_HandSolder"
 			(at 195.58 79.248 90)
 			(effects
